File: EDA-kicad/NFC.kicad_sch (KiCad schematic)
At the start: 25 parts, among them Y1 27.12Mhz

Commit message: last adjustement
Changed lines of the file:
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@@
 		(on_board yes)
 		(dnp no)
-		(property "Reference" "#3.3V010"
+		(property "Reference" "#3.3V012"
 			(at 161.544 78.232 0)
 			(effects
@@
 			(project "cm5-carrier"
 				(path "/28c5e4fe-1ec7-4477-97f0-d2ec1401fad5/bde4301f-747d-4aba-a21c-9ee44896b6bc"
-					(reference "#3.3V010")
+					(reference "#3.3V012")
 					(unit 1)
 				)
