File: EDA-kicad/cm5-carrier.kicad_sch (KiCad schematic)
At the start: 6 parts

Commit message: last adjustement
Other:
- added sheet NFC (NFC.kicad_sch)
- note added: "Icon by afif fudin from Flaticon"

Commit message: last adjustement
Parts:
- added R22, R23: 4.7k, symbol Device:R_Small
Connections:
- net DIS SCL: now also R23.2
- net DIS SDA: now also R22.2
- net VCC: now also R22.1, R23.1
- net SE050 ENA: now reaches Module1.41 (GPIO25)
- net NFC VEN: now reaches Module1.45 (GPIO24)
- net NFC INTERRUPT: now reaches Module1.49 (GPIO18)
